Commit message: upload finished week 2

File: hrwros_ws/src/hrwros_week2/urdf/hrwros_assignment1.xacro (robot description, xacro)
@@ -72,3 +72,10 @@
   </joint>
   <!-- Add your solution to assignment 1 here -->
+  <!-- extra bin -->
+  <xacro:bin_urdf prefix="bin_extra_"/>
+  <joint name="bin_extra_joint" type="fixed">
+    <parent link="world_interface" />
+    <child link="bin_extra_base_link" />
+    <origin xyz="2.05 1.8 0.0" rpy="0 0 0" />
+  </joint>
 </robot>

File: hrwros_ws/src/hrwros_week2/urdf/hrwros_assignment2.xacro (robot description, xacro)
@@ -72,3 +72,19 @@
   </joint>
   <!-- Add your solution to assignment 2 here -->
+  <material name="green">
+   <color rgba="0 0.8 0 1"/>
+  </material>
+  <link name="sphere_dummy_link">
+   <visual>
+    <geometry>
+     <sphere radius="0.4"/>
+    </geometry>
+    <material name="green"/>
+   </visual>
+  </link>
+  <joint name="sphere_dummy_joint" type="fixed">
+   <parent link="world_interface" />
+   <child link="sphere_dummy_link" />
+   <origin xyz="5.5 -5 0.4" rpy="0 0 0" />
+  </joint>
 </robot>

File: hrwros_ws/src/hrwros_week2/urdf/hrwros_assignment3.xacro (robot description, xacro)
@@ -61,9 +61,16 @@
   <joint name="robot2_pedestal_joint" type="fixed">
     <origin xyz="-7.8 -1.5 0" />
-    <parent link="world" />
+    <parent link="world_interface" />
     <child link="robot2_pedestal_link" />
   </joint>
   <!-- Update the below block for assignment 3 here -->
-  <xacro:include filename="$(find ur_description)/urdf/ur5.urdf.xacro"/>
+  <xacro:include filename="$(find hrwros_week2)/urdf/robot/lrmate200ic_macro.xacro"/>
+  <xacro:fanuc_lrmate200ic prefix="robot2_" />
+  <joint name="robot2-pedestal_joint" type="fixed">
+    <parent link="robot2_pedestal_link" />
+    <child link="robot2_base_link" />
+    <origin xyz="0 0 0.6" rpy="0 0 0" />
+  </joint>
+  <!-- <xacro:include filename="$(find ur_description)/urdf/ur5.urdf.xacro"/>
   <xacro:ur5_robot prefix="robot2_" joint_limited="true"/>
   <joint name="robot2-robot2_pedestal_joint" type="fixed">
@@ -71,4 +78,4 @@
     <child link="robot2_base_link" />
     <origin xyz="0 0 0.6" rpy="0 0 ${radians(90)}" />
-  </joint>
+  </joint> -->
 </robot>
